File: PCB/easylight.kicad_pcb (KiCad board)
At the start: 2 copper layers, 50.2 x 41.3 mm, 49 parts, among them J1 LiPo (1S/3.7V), J2 USB/PWR, J3 LEDs, J4 AVR-ISP, J8 SW4+, Q1 AO3415_C181094, Q2 AO3415_C181094, SW0 SPEF110100, SW1 TS-1187A-B-A-B, SW2 TS-1187A-B-A-B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

Commit message: add more labels, replace broken SOT23 with generic part, update version, cleanup part descriptions
Parts:
- C8: footprint Capacitor_SMD:C_1206_3216Metric_Pad1.42x1.75mm_HandSolder -> Capacitor_SMD:C_1206_3216Metric_Pad1.33x1.80mm_HandSolder
- J1: value LiPo (1S/3.7V) -> LiPo (3.7V)
- Q1, Q2: footprint lcsc:SOT-23-3_L2.9-W1.3-P1.90-LS2.4-BR -> Package_TO_SOT_SMD:SOT-23-3
- moved Q1 0.27 mm to (58.4, 56.8), turned to 180 degrees
- turned Q2 to 180 degrees
Routing:
- net GND: vias 18 -> 17
Other:
- board text added: "CHRG"
- board text added: "D1"
- board text added: "D2"
- board text added: "LEDs"
- board text added: "LiPo (3.7V)"
- board text added: "USB/PWR"

Commit message: use generic part for SOIC-8, ignore another lib warning
Parts:
- U3: footprint LCSC:SOIC-8_L4.9-W3.9-P1.27-LS6.0-BL-EP3.3-1 -> Package_SO:SOIC-8-1EP_3.9x4.9mm_P1.27mm_EP2.514x3.2mm
- turned U3 to -90 degrees
Changed lines of the file:
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@@
     )
   )
-  (footprint "LCSC:SOIC-8_L4.9-W3.9-P1.27-LS6.0-BL-EP3.3-1" (layer "F.Cu")
-    (at 50.805 52.525 180)
+  (footprint "Package_SO:SOIC-8-1EP_3.9x4.9mm_P1.27mm_EP2.514x3.2mm" (layer "F.Cu")
+    (at 50.8 52.525 -90)
+    (descr "SOIC, 8 Pin (https://www.renesas.com/eu/en/www/doc/datasheet/hip2100.pdf#page=13), generated with kicad-footprint-generator ipc_gullwing_generator.py")
+    (tags "SOIC SO")
     (property "JLC Part" "Extended Part")
     (property "LCSC Part" "C2760005")
@@
     (property "Sheetname" "")
     (attr smd)
-    (fp_text reference "U3" (at -3.17 0 270) (layer "F.SilkS")
-      (effects (font (size 1 1) (thickness 0.15)))
-    )
-    (fp_text value "XB8089D0" (at 0 6.72 180) (layer "F.Fab")
-      (effects (font (size 1 1) (thickness 0.15)))
-    )
-    (fp_text user "${REFERENCE}" (at 0 0 180) (layer "F.Fab")
-      (effects (font (size 1 1) (thickness 0.15)))
-    )
-    (fp_line (start 2.53 -1.52) (end 2.53 1.52) (layer "F.SilkS") (width 0.15))
-    (fp_line (start -2.53 -1.52) (end 2.53 -1.52) (layer "F.SilkS") (width 0.15))
-    (fp_line (start -2.53 1.52) (end -2.53 -1.52) (layer "F.SilkS") (width 0.15))
-    (fp_line (start 2.53 1.52) (end -2.53 1.52) (layer "F.SilkS") (width 0.15))
-    (fp_circle (center -2.16 1.14) (end -2.01 1.14) (layer "F.SilkS") (width 0.3) (fill none))
-    (fp_circle (center -2.66 2.72) (end -2.51 2.72) (layer "F.SilkS") (width 0.3) (fill none))
-    (fp_circle (center -1.9 3.4) (end -1.75 3.4) (layer "Cmts.User") (width 0.3) (fill none))
-    (fp_circle (center -2.45 3) (end -2.42 3) (layer "F.Fab") (width 0.06) (fill none))
-    (pad "1" smd oval locked (at -1.9 2.72 180) (size 0.6 1.94) (layers "F.Cu" "F.Paste" "F.Mask")
+    (fp_text reference "U3" (at 0 -3.4 -90) (layer "F.SilkS")
+      (effects (font (size 1 1) (thickness 0.15)))
+    )
+    (fp_text value "XB8089D0" (at 0 3.4 -90) (layer "F.Fab")
+      (effects (font (size 1 1) (thickness 0.15)))
+    )
+    (fp_text user "${REFERENCE}" (at 0 0 -90) (layer "F.Fab")
+      (effects (font (size 0.98 0.98) (thickness 0.15)))
+    )
+    (fp_line (start 0 2.56) (end -1.95 2.56) (layer "F.SilkS") (width 0.12))
+    (fp_line (start 0 -2.56) (end 1.95 -2.56) (layer "F.SilkS") (width 0.12))
+    (fp_line (start 0 2.56) (end 1.95 2.56) (layer "F.SilkS") (width 0.12))
+    (fp_line (start 0 -2.56) (end -3.45 -2.56) (layer "F.SilkS") (width 0.12))
+    (fp_line (start 3.7 2.7) (end 3.7 -2.7) (layer "F.CrtYd") (width 0.05))
+    (fp_line (start -3.7 -2.7) (end -3.7 2.7) (layer "F.CrtYd") (width 0.05))
+    (fp_line (start 3.7 -2.7) (end -3.7 -2.7) (layer "F.CrtYd") (width 0.05))
+    (fp_line (start -3.7 2.7) (end 3.7 2.7) (layer "F.CrtYd") (width 0.05))
+    (fp_line (start 1.95 2.45) (end -1.95 2.45) (layer "F.Fab") (width 0.1))
+    (fp_line (start -1.95 2.45) (end -1.95 -1.475) (layer "F.Fab") (width 0.1))
+    (fp_line (start -1.95 -1.475) (end -0.975 -2.45) (layer "F.Fab") (width 0.1))
+    (fp_line (start 1.95 -2.45) (end 1.95 2.45) (layer "F.Fab") (width 0.1))
+    (fp_line (start -0.975 -2.45) (end 1.95 -2.45) (layer "F.Fab") (width 0.1))
+    (pad "" smd roundrect (at -0.63 0.8 270) (size 1.01 1.29) (layers "F.Paste") (roundrect_rratio 0.247525))
+    (pad "" smd roundrect (at 0.63 -0.8 270) (size 1.01 1.29) (layers "F.Paste") (roundrect_rratio 0.247525))
+    (pad "" smd roundrect (at 0.63 0.8 270) (size 1.01 1.29) (layers "F.Paste") (roundrect_rratio 0.247525))
+    (pad "" smd roundrect (at -0.63 -0.8 270) (size 1.01 1.29) (layers "F.Paste") (roundrect_rratio 0.247525))
+    (pad "1" smd roundrect (at -2.6375 -1.905 270) (size 1.625 0.6) (layers "F.Cu" "F.Paste" "F.Mask") (roundrect_rratio 0.25)
       (net 2 "GND") (pinfunction "VM") (pintype "power_in"))
-    (pad "2" smd oval locked (at -0.63 2.72 180) (size 0.6 1.94) (layers "F.Cu" "F.Paste" "F.Mask")
+    (pad "2" smd roundrect (at -2.6375 -0.635 270) (size 1.625 0.6) (layers "F.Cu" "F.Paste" "F.Mask") (roundrect_rratio 0.25)
       (net 2 "GND") (pinfunction "VM") (pintype "power_in"))
-    (pad "3" smd oval locked (at 0.64 2.72 180) (size 0.6 1.94) (layers "F.Cu" "F.Paste" "F.Mask")
+    (pad "3" smd roundrect (at -2.6375 0.635 270) (size 1.625 0.6) (layers "F.Cu" "F.Paste" "F.Mask") (roundrect_rratio 0.25)
       (net 2 "GND") (pinfunction "VM") (pintype "power_in"))
-    (pad "4" smd oval locked (at 1.9 2.72 180) (size 0.6 1.94) (layers "F.Cu" "F.Paste" "F.Mask")
+    (pad "4" smd roundrect (at -2.6375 1.905 270) (size 1.625 0.6) (layers "F.Cu" "F.Paste" "F.Mask") (roundrect_rratio 0.25)
       (net 2 "GND") (pinfunction "VM") (pintype "power_in"))
-    (pad "5" smd oval locked (at 1.9 -2.72 180) (size 0.6 1.94) (layers "F.Cu" "F.Paste" "F.Mask")
+    (pad "5" smd roundrect (at 2.6375 1.905 270) (size 1.625 0.6) (layers "F.Cu" "F.Paste" "F.Mask") (roundrect_rratio 0.25)
       (net 6 "-BATT") (pinfunction "GND") (pintype "power_in"))
-    (pad "6" smd oval locked (at 0.64 -2.72 180) (size 0.6 1.94) (layers "F.Cu" "F.Paste" "F.Mask")
+    (pad "6" smd roundrect (at 2.6375 0.635 270) (size 1.625 0.6) (layers "F.Cu" "F.Paste" "F.Mask") (roundrect_rratio 0.25)
       (net 7 "Net-(C4-Pad1)") (pinfunction "VDD") (pintype "power_out"))
-    (pad "7" smd oval locked (at -0.63 -2.72 180) (size 0.6 1.94) (layers "F.Cu" "F.Paste" "F.Mask")
+    (pad "7" smd roundrect (at 2.6375 -0.635 270) (size 1.625 0.6) (layers "F.Cu" "F.Paste" "F.Mask") (roundrect_rratio 0.25)
       (net 6 "-BATT") (pinfunction "GND") (pintype "power_in"))
-    (pad "8" smd oval locked (at -1.9 -2.72 180) (size 0.6 1.94) (layers "F.Cu" "F.Paste" "F.Mask")
+    (pad "8" smd roundrect (at 2.6375 -1.905 270) (size 1.625 0.6) (layers "F.Cu" "F.Paste" "F.Mask") (roundrect_rratio 0.25)
       (net 6 "-BATT") (pinfunction "GND") (pintype "power_in"))
-    (pad "9" smd rect locked (at 0 0 180) (size 3.3 2.4) (layers "F.Cu" "F.Paste" "F.Mask")
+    (pad "9" smd rect (at 0 0 270) (size 2.514 3.2) (layers "F.Cu" "F.Mask")
       (net 6 "-BATT") (pinfunction "EP") (pintype "power_in"))
-    (model "D:/Kreativ/PCB/KiCad/lcsc.3dshapes/SOIC-8_L4.9-W3.9-P1.27-LS6.0-BL-EP3.3-1.wrl"
-      (offset (xyz 0 -0.08 -0))
+    (model "${KICAD6_3DMODEL_DIR}/Package_SO.3dshapes/SOIC-8-1EP_3.9x4.9mm_P1.27mm_EP2.35x2.35mm.step"
+      (offset (xyz 0 0 0))
       (scale (xyz 1 1 1))
       (rotate (xyz 0 0 0))
@@
   (via (at 64.135 48.895) (size 0.8) (drill 0.4) (layers "F.Cu" "B.Cu") (net 2))
   (via (at 41.275 72.39) (size 0.8) (drill 0.4) (layers "F.Cu" "B.Cu") (net 2))
-  (via (at 62.23 66.52) (size 0.8) (drill 0.4) (layers "F.Cu" "B.Cu") (net 2))
+  (via (at 62.23 66.294) (size 0.8) (drill 0.4) (layers "F.Cu" "B.Cu") (net 2))
   (segment (start 42.7225 65.5825) (end 43.18 66.04) (width 0.5) (layer "F.Cu") (net 3))
   (segment (start 42.7225 64.135) (end 42.7225 65.5825) (width 0.5) (layer "F.Cu") (net 3))
@@
   (segment (start 56.89 65.085) (end 56.89 65.78) (width 0.5) (layer "F.Cu") (net 14))
   (via (at 57.15 66.04) (size 0.8) (drill 0.4) (layers "F.Cu" "B.Cu") (net 14))
-  (segment (start 57.949999 65.240001) (end 65.875001 65.240001) (width 0.5) (layer "B.Cu") (net 14))
-  (segment (start 65.875001 65.240001) (end 66.675 66.04) (width 0.5) (layer "B.Cu") (net 14))
-  (segment (start 57.15 66.04) (end 57.949999 65.240001) (width 0.5) (layer "B.Cu") (net 14))
+  (segment (start 65.405 64.77) (end 66.675 66.04) (width 0.5) (layer "B.Cu") (net 14))
+  (segment (start 57.15 66.04) (end 58.42 64.77) (width 0.5) (layer "B.Cu") (net 14))
+  (segment (start 58.42 64.77) (end 65.405 64.77) (width 0.5) (layer "B.Cu") (net 14))
   (segment (start 66.675 57.785) (end 66.675 60.96) (width 0.5) (layer "F.Cu") (net 15))
   (segment (start 75.845001 69.028001) (end 74.943001 69.930001) (width 0.5) (layer "B.Cu") (net 15))

Commit message: improve fills, add qr code, improve silkscreen labels
Parts:
- added G2: LOGO, ModischFabrications:MF_QR_7mm, B.Cu at (64.1, 77.5)
- L1: footprint ModischFabrications:mpc_logo_10mm -> ModischFabrications:mpc_logo_5mm
- moved L2 27.3 mm to (73.7, 77.5)
- moved SYM1 13.4 mm to (54.6, 78.7)
- moved G1 8.26 mm to (48.3, 78.7)
- moved L1 1.42 mm to (75.6, 52.1)
Routing:
- net Net-(D3-Pad1): track 24.2 -> 6.47 mm
- added copper zone on F.Cu, net Net-(D3-Pad1)
Other:
- board text added: "${TITLE} v${REVISION} ${ISSUE_DATE}"
- board text added: "Modisch Popp Creations"
- board text removed: "${ISSUE_DATE} v${REVISION}"
- board text removed: "${TITLE}"
- board text removed: "© Modisch Popp Creations"
